File: Engine/Engine.kicad_pcb (KiCad board)
At the start: 4 copper layers, 18 x 24 mm, 33 parts, among them J1 Conn_01x02, J2 Conn_01x02, J3 Conn_01x02, J4 Conn_01x02, J5 Conn_01x03, J6 TC_2030_NL_STLINK, Q1 FDN335N, Q2 FDN335N, U1 MCP1755T-3302E/OT, U2 STM32L011KxUx, U3 DRV8220DSGR, U4 TLV9041IDBVR

Commit message: New smaller version
Parts:
- removed Q2: FDN335N, U_IC:SOT23_3
- removed U4: TLV9041IDBVR, U_IC:SOT23_5
- added C12: C_0402, C_Capacitor:C_0402, F.Cu at (85.2, 81.1)
- added J10: Pad_4x2, N-NonPart:MountingPad_2.0x2.0mm, B.Cu at (91.3, 90.6)
- added J11: Pad_4x2, N-NonPart:MountingPad_2.0x2.0mm, B.Cu at (89.0, 90.6)
- added J12: TC_2030_NL_STLINK, N-NonPart:TagConnect_2030_NL, F.Cu at (92.6, 83.7)
- added J7: Pad_4x2, N-NonPart:MountingPad_2.0x2.0mm, B.Cu at (79.1, 83.2)
- added J8: Pad_4x2, N-NonPart:MountingPad_2.0x2.0mm, B.Cu at (79.1, 85.5)
- added J9: Pad_4x2, N-NonPart:MountingPad_2.0x2.0mm, B.Cu at (93.6, 90.6)
- added R9: R_0402, R_Resistor:R_0402, F.Cu at (90.3, 84.6)
- J1, J2, J3, J4: value Conn_01x02 -> Pad_4x2; footprint Connector_PinHeader_2.54mm:PinHeader_1x02_P2.54mm_Vertical -> N-NonPart:MountingPad_2.0x2.0mm; moved to B.Cu
- J5: value Conn_01x03 -> Pad_4x2; footprint Connector_PinHeader_2.54mm:PinHeader_1x03_P2.54mm_Vertical -> N-NonPart:MountingPad_2.0x2.0mm; moved to B.Cu
- J6: value TC_2030_NL_STLINK -> Pad_4x2; footprint N-NonPart:TagConnect_2030_NL -> N-NonPart:MountingPad_2.0x2.0mm; moved to B.Cu
- Q1: value FDN335N -> DMN601VK-7; footprint U_IC:SOT23_3 -> U_IC:SOT563
- R2: value R_0603 -> R_0402; footprint R_Resistor:R_0603 -> R_Resistor:R_0402
- R4: value R_0402 -> R_0603; footprint R_Resistor:R_0402 -> R_Resistor:R_0603
- moved R4 51.3 mm to (80.3, 82.8), turned to 180 degrees
- moved J1 49.8 mm to (83.5, 78.5)
- moved R2 48.9 mm to (80.7, 89.8)
- moved J6 48.7 mm to (79.1, 80.8)
- moved C6 47.5 mm to (89.1, 90.2)
- moved J3 45.9 mm to (79.1, 87.8), turned to 180 degrees
- moved D1 45.8 mm to (85.2, 78.8), turned to 180 degrees
- moved C1 45.7 mm to (83.2, 89.8)
- moved C5 45.6 mm to (87.6, 89.8)
- moved U1 45.6 mm to (85.4, 90.1)
- moved C7 43.9 mm to (91.1, 90.2)
- moved J4 43.9 mm to (79.1, 90.1), turned to 180 degrees
- moved Q1 43.4 mm to (80.4, 80.5)
- moved C3 42.7 mm to (90.1, 87.3)
- moved U2 42.6 mm to (86.4, 84.8)
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Connections:
- C10 pad 1: Net-(C10-Pad1) -> /Input/RX_OUT+
- C10 pad 2: Net-(C10-Pad2) -> GND
- C11 pad 1: +12V -> GND
- C11 pad 2: GND -> /Input/RX_OUT-
- J1 pad 1: /Input/IN_A -> /Input/IN_B
- J2 pad 1: /Outputs/MTR_OUT_A -> /Input/IN_A
- J3 pad 1: /Outputs/LED_1_+ -> /Outputs/MTR_OUT_A
- J4 pad 1: /Outputs/LED_2_+ -> /Outputs/MTR_OUT_B
- J5 pad 1: +3V3 -> /Outputs/LED_1+
- J6 pad 1: +3V3 -> /Outputs/LED_1-
- Q1 pad 1: /MCU/LED_1 -> GND
- Q1 pad 2: GND -> /MCU/LED_1
- Q1 pad 3: /Outputs/LED_1_- -> /Outputs/LED_2-
- R2 pad 1: +12V -> /MCU/LED_DBG
- R2 pad 2: /Outputs/LED_1_+ -> Net-(DS1-Pad2)
- R3 pad 2: /Outputs/LED_2_+ -> /Outputs/LED_1+
- R4 pad 1: /Input/IN_A -> +12V
- R4 pad 2: Net-(C10-Pad1) -> /Outputs/LED_2+
- R5 pad 1: /Input/IN_B -> /Input/IN_A
- R5 pad 2: Net-(C10-Pad2) -> /Input/RX_OUT+
- R6 pad 1: Net-(C10-Pad1) -> /Input/IN_B
- R6 pad 2: GND -> /Input/RX_OUT-
- R7 pad 1: GND -> /Input/RX_OUT+
- R7 pad 2: Net-(C10-Pad2) -> GND
- R8 pad 1: /MCU/LED_DBG -> GND
- R8 pad 2: Net-(DS1-Pad2) -> /Input/RX_OUT-
- U2 pad 19: /MCU/AUX_TX -> unconnected-(U2-Pad19)
- U2 pad 20: unconnected-(U2-Pad20) -> /Input/RX_FB
- U2 pad 22: unconnected-(U2-Pad22) -> /Input/RX_FB
- U2 pad 26: unconnected-(U2-Pad26) -> /Input/RX_OUT-
- U2 pad 27: unconnected-(U2-Pad27) -> /Input/RX_OUT+
- U2 pad 29: unconnected-(U2-Pad29) -> /MCU/AUX_TX
- U2 pad 30: /Input/IN_RX -> unconnected-(U2-Pad30)
- U2 pad 6: /MCU/MTR_A -> /MCU/MTR_nSLEEP
- U2 pad 7: /MCU/MTR_B -> /MCU/MTR_MODE
- U2 pad 8: /MCU/MTR_nSLEEP -> /MCU/MTR_A
- U2 pad 9: /MCU/MTR_MODE -> /MCU/MTR_B
Routing:
- net /MCU/SWCLK: track 15.7 -> 4.53 mm
- net /Input/IN_RX: track 10.3 -> 0.00 mm, vias 2 -> 0
- net /Input/RX_OUT+: track 0.00 -> 9.93 mm, vias 0 -> 2
- net /Outputs/LED_2-: track 0.00 -> 8.68 mm, vias 0 -> 1
- net /MCU/SWDIO: track 12.9 -> 5.34 mm
- net /Input/RX_OUT-: track 0.00 -> 6.59 mm
- net /MCU/LED_1: track 11.4 -> 4.88 mm, vias 2 -> 0
- net /MCU/NRST: track 12.9 -> 18.4 mm
- net /MCU/MTR_MODE: track 8.25 -> 2.95 mm, vias 2 -> 0
- net /MCU/MTR_nSLEEP: track 7.63 -> 2.95 mm, vias 2 -> 0
- net /Input/IN_A: track 6.70 -> 2.55 mm, vias 0 -> 3
- net +3V3: track 11.5 -> 7.65 mm, vias 8 -> 9
- net /Input/IN_B: track 7.01 -> 10.5 mm, vias 1 -> 4
- net Net-(C10-Pad2): track 3.45 -> 0.00 mm
- net Net-(C10-Pad1): track 3.42 -> 0.00 mm
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- added copper zone on B.Cu, net /Input/IN_A
- added copper zone on F.Cu, net /Input/IN_A
- added copper zone on F.Cu, net /Input/IN_B
Other:
- board size 18 x 24 mm -> 17.3 x 15.3 mm
- board text added: "A"
- board text added: "B"
- board text added: "IN"
- board text added: "L1"
- board text added: "L2"
- board text added: "MTR"
- board text removed: "LED1"
- board text removed: "LED2"
- board text removed: "MOTOR"
- board text removed: "RAIL"
