File: Engine/Engine.kicad_sch (KiCad schematic)
At the start: 5 parts, among them J1 Conn_01x02, J2 Conn_01x02, J3 Conn_01x02, J4 Conn_01x02, J5 Conn_01x03

Commit message: New smaller version
Parts:
- removed J1, J2, J3, J4: Conn_01x02, Connector_PinHeader_2.54mm:PinHeader_1x02_P2.54mm_Vertical, symbol Connector_Generic:Conn_01x02
- removed J5: Conn_01x03, Connector_PinHeader_2.54mm:PinHeader_1x03_P2.54mm_Vertical, symbol Connector_Generic:Conn_01x03
- added J1, J10, J11, J2, J3, J4, J5, J6, J7, J8, J9: Pad_4x2, N-NonPart:MountingPad_2.0x2.0mm, symbol J_Connector:Pad_4x2
Connections:
- net +3V3: now also J9.1
- net GND: now also J11.1
- net Input/IN_A: now also J2.1
- net Input/IN_B: now also J1.1
- net MCU/AUX_TX: now also J10.1
- net Outputs/MTR_OUT_A: now also J3.1
- net Outputs/MTR_OUT_B: now also J4.1
- new net Outputs/LED_1+: J5.1
- new net Outputs/LED_1-: J6.1
- new net Outputs/LED_2+: J7.1
- new net Outputs/LED_2-: J8.1
Other:
- sheet Input ports: added RX_FB, RX_OUT+, RX_OUT-; removed IN_RX
- sheet MCU ports: added RX_IN+, RX_IN-, RX_OUT; removed IN_RX
- sheet Outputs ports: added LED_1+, LED_1-, LED_2+, LED_2-; removed LED_1_+, LED_1_-, LED_2_+, LED_2_-
