File: Engine/input.kicad_sch (KiCad schematic)
At the start: 8 parts, among them U4 TLV9041IDBVR

Commit message: New smaller version
Parts:
- removed U4: TLV9041IDBVR, U_IC:SOT23_5, symbol U_Basic:TLV9041IDBVR
- added C10: C_0402, C_Capacitor:C_0402, symbol C_Capacitor:C_0402
- added R9: R_0402, R_Resistor:R_0402, symbol R_Resistor:R_0402
- R7: renamed from R6; Resistance 1K -> 10K
- R8: renamed from R7; Resistance 1K -> 10K
- renumbered C10 to C11, C11 to C12, R4 to R5, R5 to R6
Connections:
- net GND: now also C11.1, C10.2
- net RX_OUT+: now reaches R5.2, R7.1
- net RX_OUT+: now also C10.1, R9.1; no longer C11.1
- net RX_OUT-: now reaches C11.2, R6.2, R8.2
- new net RX_FB: R9.2
Other:
- moved on the sheet: C11, R6, R8
