File: Engine/outputs.kicad_sch (KiCad schematic)
At the start: 7 parts, among them Q1 FDN335N, Q2 FDN335N, U3 DRV8220DSGR

Commit message: New smaller version
Parts:
- removed Q1, Q2: FDN335N, U_IC:SOT23_3, symbol Q_MOSFET:FDN335N
- added Q1: DMN601VK-7, U_IC:SOT563, symbol Q_MOSFET:DMN601VK-7
- renumbered R2 to R3, R3 to R4
Connections:
- net GND: now also Q1.1 (S), Q1.4 (S)
- net LED_1: now also Q1.2 (G)
- net LED_2: now also Q1.5 (G)
- net LED_1_+ renamed LED_1+
- net LED_2_+ renamed LED_2+
- new net LED_1-: Q1.6 (D)
- new net LED_2-: Q1.3 (D)
Changed lines of the file:
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@@
     (effects (font (size 1.27 1.27)) (justify right))
   )
-  (hierarchical_label "LED_2_-" (shape output) (at 92.71 138.43 0)
-    (effects (font (size 1.27 1.27)) (justify left))
-  )
-  (hierarchical_label "LED_1_+" (shape output) (at 92.71 93.98 0)
+  (hierarchical_label "LED_2-" (shape output) (at 92.71 138.43 0)
+    (effects (font (size 1.27 1.27)) (justify left))
+  )
+  (hierarchical_label "LED_1+" (shape output) (at 92.71 93.98 0)
     (effects (font (size 1.27 1.27)) (justify left))
   )
@@
     (effects (font (size 1.27 1.27)) (justify left))
   )
-  (hierarchical_label "LED_2_+" (shape output) (at 92.71 133.35 0)
+  (hierarchical_label "LED_2+" (shape output) (at 92.71 133.35 0)
     (effects (font (size 1.27 1.27)) (justify left))
   )
@@
     (effects (font (size 1.27 1.27)) (justify left))
   )
-  (hierarchical_label "LED_1_-" (shape output) (at 92.71 99.06 0)
+  (hierarchical_label "LED_1-" (shape output) (at 92.71 99.06 0)
     (effects (font (size 1.27 1.27)) (justify left))
   )
   (symbol (lib_id "power:GND") (at 90.17 151.13 0) (unit 1)
     (in_bom yes) (on_board yes) (fields_autoplaced)
-    (property "Reference" "#PWR018" (id 0) (at 90.17 157.48 0)
+    (property "Reference" "#PWR019" (id 0) (at 90.17 157.48 0)
       (effects (font (size 1.27 1.27)) hide)
     )
@@
   (symbol (lib_id "power:GND") (at 90.17 111.76 0) (unit 1)
     (in_bom yes) (on_board yes) (fields_autoplaced)
-    (property "Reference" "#PWR016" (id 0) (at 90.17 118.11 0)
+    (property "Reference" "#PWR017" (id 0) (at 90.17 118.11 0)
       (effects (font (size 1.27 1.27)) hide)
     )
@@
     (pin "2")
   )
-  (symbol (lib_id "Q_MOSFET:FDN335N") (at 90.17 105.41 0) (unit 1)
-    (in_bom yes) (on_board yes) (fields_autoplaced)
-    (property "Reference" "Q1" (id 0) (at 92.075 104.9079 0)
-      (effects (font (size 1.27 1.27)) (justify left))
-    )
-    (property "Value" "FDN335N" (id 1) (at 92.075 107.0275 0)
-      (effects (font (size 0.6096 0.6096)) (justify left))
-    )
-    (property "Footprint" "U_IC:SOT23_3" (id 2) (at 99.06 107.315 0)
-      (effects (font (size 1.27 1.27)) hide)
-    )
-    (property "Datasheet" "https://www.onsemi.com/pdf/datasheet/fdn335n-d.pdf" (id 3) (at 88.9 118.11 0)
-      (effects (font (size 1.27 1.27)) hide)
-    )
-    (pin "1")
-    (pin "2")
-    (pin "3")
+  (symbol (lib_id "Q_MOSFET:DMN601VK-7") (at 90.17 105.41 0) (unit 1)
+    (in_bom yes) (on_board yes) (fields_autoplaced)
+    (property "Reference" "Q1" (id 0) (at 92.075 104.5015 0)
+      (effects (font (size 1.27 1.27)) (justify left))
+    )
+    (property "Value" "DMN601VK-7" (id 1) (at 92.075 107.2766 0)
+      (effects (font (size 1.27 1.27)) (justify left))
+    )
+    (property "Footprint" "U_IC:SOT563" (id 2) (at 97.79 109.22 0)
+      (effects (font (size 1.27 1.27)) hide)
+    )
+    (property "Datasheet" "" (id 3) (at 90.17 105.41 0)
+      (effects (font (size 1.27 1.27)) hide)
+    )
+    (pin "1")
+    (pin "2")
+    (pin "6")
   )
   (symbol (lib_id "U_Driver:DRV8220DSGR") (at 101.6 54.61 0) (unit 1)
@@
     (pin "9")
   )
-  (symbol (lib_id "Q_MOSFET:FDN335N") (at 90.17 144.78 0) (unit 1)
-    (in_bom yes) (on_board yes) (fields_autoplaced)
-    (property "Reference" "Q2" (id 0) (at 92.075 144.2779 0)
-      (effects (font (size 1.27 1.27)) (justify left))
-    )
-    (property "Value" "FDN335N" (id 1) (at 92.075 146.3975 0)
-      (effects (font (size 0.6096 0.6096)) (justify left))
-    )
-    (property "Footprint" "U_IC:SOT23_3" (id 2) (at 99.06 146.685 0)
-      (effects (font (size 1.27 1.27)) hide)
-    )
-    (property "Datasheet" "https://www.onsemi.com/pdf/datasheet/fdn335n-d.pdf" (id 3) (at 88.9 157.48 0)
-      (effects (font (size 1.27 1.27)) hide)
-    )
-    (pin "1")
-    (pin "2")
+  (symbol (lib_id "Q_MOSFET:DMN601VK-7") (at 90.17 144.78 0) (unit 2)
+    (in_bom yes) (on_board yes) (fields_autoplaced)
+    (property "Reference" "Q1" (id 0) (at 92.075 143.8715 0)
+      (effects (font (size 1.27 1.27)) (justify left))
+    )
+    (property "Value" "DMN601VK-7" (id 1) (at 92.075 146.6466 0)
+      (effects (font (size 1.27 1.27)) (justify left))
+    )
+    (property "Footprint" "U_IC:SOT563" (id 2) (at 97.79 148.59 0)
+      (effects (font (size 1.27 1.27)) hide)
+    )
+    (property "Datasheet" "" (id 3) (at 90.17 144.78 0)
+      (effects (font (size 1.27 1.27)) hide)
+    )
     (pin "3")
+    (pin "4")
+    (pin "5")
   )
   (symbol (lib_id "power:+12V") (at 90.17 123.19 0) (unit 1)
     (in_bom yes) (on_board yes) (fields_autoplaced)
-    (property "Reference" "#PWR017" (id 0) (at 90.17 127 0)
+    (property "Reference" "#PWR018" (id 0) (at 90.17 127 0)
       (effects (font (size 1.27 1.27)) hide)
     )
@@
   (symbol (lib_id "R_Resistor:R_0603") (at 90.17 128.27 0) (unit 1)
     (in_bom yes) (on_board yes) (fields_autoplaced)
-    (property "Reference" "R3" (id 0) (at 91.821 126.6042 0)
+    (property "Reference" "R4" (id 0) (at 91.821 126.6042 0)
       (effects (font (size 1.27 1.27)) (justify left))
     )
@@
   (symbol (lib_id "power:+12V") (at 90.17 83.82 0) (unit 1)
     (in_bom yes) (on_board yes) (fields_autoplaced)
-    (property "Reference" "#PWR015" (id 0) (at 90.17 87.63 0)
+    (property "Reference" "#PWR016" (id 0) (at 90.17 87.63 0)
       (effects (font (size 1.27 1.27)) hide)
     )
@@
   (symbol (lib_id "power:+12V") (at 120.142 45.72 0) (unit 1)
     (in_bom yes) (on_board yes) (fields_autoplaced)
-    (property "Reference" "#PWR019" (id 0) (at 120.142 49.53 0)
+    (property "Reference" "#PWR020" (id 0) (at 120.142 49.53 0)
       (effects (font (size 1.27 1.27)) hide)
     )
@@
   (symbol (lib_id "R_Resistor:R_0603") (at 90.17 88.9 0) (unit 1)
     (in_bom yes) (on_board yes) (fields_autoplaced)
-    (property "Reference" "R2" (id 0) (at 91.821 87.2342 0)
+    (property "Reference" "R3" (id 0) (at 91.821 87.2342 0)
       (effects (font (size 1.27 1.27)) (justify left))
     )
@@
   (symbol (lib_id "power:GND") (at 120.142 66.04 0) (unit 1)
     (in_bom yes) (on_board yes) (fields_autoplaced)
-    (property "Reference" "#PWR020" (id 0) (at 120.142 72.39 0)
-      (effects (font (size 1.27 1.27)) hide)
-    )
+    (property "Reference" "#PWR021" (id 0) (at 120.142 72.39 0)
+      (effects (font (size 1.27 1.27)) hide)
+    )
